File: vca_3360/3360 VCA.sch (KiCad schematic (older format))
At the start: 51 parts, among them J1 Power in, J2 Input?, J3 CV1 In, J4 Input2, J5 CV2 In, J6 LED1, J7 LED2, J8 OUTPUT1, J9 OUTPUT2, Q1 2N3904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

Commit message: attenuverter and 3340 schematics
Parts:
- C1, C2: value CP_Small -> 10uf
- J2: value Input? -> Input1
Changed lines of the file:
@@
 P 3550 3550
 F 0 "J2" H 3658 3731 50  0000 C CNN
-F 1 "Input?" H 3658 3640 50  0000 C CNN
+F 1 "Input1" H 3658 3640 50  0000 C CNN
 F 2 "Connector_PinSocket_2.54mm:PinSocket_1x02_P2.54mm_Vertical" H 3550 3550 50  0001 C CNN
 F 3 "~" H 3550 3550 50  0001 C CNN
@@
 P 2550 8200
 F 0 "C1" H 2638 8246 50  0000 L CNN
-F 1 "CP_Small" H 2638 8155 50  0000 L CNN
+F 1 "10uf" H 2638 8155 50  0000 L CNN
 F 2 "Capacitor_THT:CP_Radial_D5.0mm_P2.00mm" H 2550 8200 50  0001 C CNN
 F 3 "~" H 2550 8200 50  0001 C CNN
@@
 P 2550 8650
 F 0 "C2" H 2638 8696 50  0000 L CNN
-F 1 "CP_Small" H 2638 8605 50  0000 L CNN
+F 1 "10uf" H 2638 8605 50  0000 L CNN
 F 2 "Capacitor_THT:CP_Radial_D5.0mm_P2.00mm" H 2550 8650 50  0001 C CNN
 F 3 "~" H 2550 8650 50  0001 C CNN
