File: vco_3340/vco_3340.sch (KiCad schematic (older format))
At the start: 42 parts

Commit message: add pcb layout for 3340
Parts:
- added C5, C6, C7: 10uf, Capacitor_THT:CP_Radial_D5.0mm_P2.00mm, symbol Device:CP_Small
- C1, C2, C3, C4: renamed from C?; footprint (none) -> Capacitor_THT:C_Disc_D5.0mm_W2.5mm_P5.00mm
- J1, J2, J3: renamed from J?; footprint (none) -> Connector_PinHeader_2.54mm:PinHeader_1x02_P2.54mm_Vertical
- J4: renamed from J?; value 1v/oct in -> PWM; footprint (none) -> Connector_PinHeader_2.54mm:PinHeader_1x02_P2.54mm_Vertical
- J5: renamed from J?; footprint (none) -> Connector_PinHeader_2.54mm:PinHeader_1x03_P2.54mm_Vertical
- J6: renamed from J?; value Conn_01x04_Male -> Power In; footprint (none) -> Connector_PinHeader_2.54mm:PinHeader_1x04_P2.54mm_Vertical
- J7: renamed from J?; value Conn_01x02_Male -> Pulse Out; footprint (none) -> Connector_PinHeader_2.54mm:PinHeader_1x02_P2.54mm_Vertical
- J8: renamed from J?; value Conn_01x02_Male -> Saw Out; footprint (none) -> Connector_PinHeader_2.54mm:PinHeader_1x02_P2.54mm_Vertical
- J9: renamed from J?; value Conn_01x02_Male -> Tri Out; footprint (none) -> Connector_PinHeader_2.54mm:PinHeader_1x02_P2.54mm_Vertical
- R1, R10, R11, R12, R13, R14, R15, R16, R2, R3, R4, R5, R6, R7, R8, R9: renamed from R?; footprint (none) -> Resistor_THT:R_Axial_DIN0207_L6.3mm_D2.5mm_P7.62mm_Horizontal
- RV1, RV2: renamed from RV?; footprint (none) -> Connector_PinHeader_2.54mm:PinHeader_1x03_P2.54mm_Vertical
- RV3: renamed from RV?; value R_POT -> Pulse Width; footprint (none) -> Connector_PinHeader_2.54mm:PinHeader_1x03_P2.54mm_Vertical
- RV4, RV5: renamed from RV?; footprint (none) -> Potentiometer_THT:Potentiometer_Runtron_RM-065_Vertical
- U1: renamed from U?; footprint (none) -> Package_DIP:DIP-8_W7.62mm_Socket
- U2: renamed from U?; footprint (none) -> Package_DIP:DIP-16_W7.62mm_Socket
- U3: renamed from U?; footprint (none) -> Package_DIP:DIP-14_W7.62mm_Socket
Connections:
- net +12V: now also J6.1 (Pin_1), C5.1
- net +5V: now also J6.4 (Pin_4), C7.1
- net -12V: now also J6.3 (Pin_3), C6.2
- net GND: now also J6.2 (Pin_2), C5.2, C6.1, C7.2

Commit message: 3360 stencil and 3340 fixes
Parts:
- added C8: 1nf, Capacitor_THT:C_Disc_D5.0mm_W2.5mm_P5.00mm, symbol Device:C_Small
- added R17: 470R, Resistor_THT:R_Axial_DIN0207_L6.3mm_D2.5mm_P7.62mm_Horizontal, symbol Device:R
- added R18: 100K, Resistor_THT:R_Axial_DIN0207_L6.3mm_D2.5mm_P7.62mm_Horizontal, symbol Device:R
Connections:
- net GND: now also C8.1
- net at R10.1, U2.15 (VFCI): now also R17.2, R18.1; no longer U1.6 (-), U1.7
- new net: C8.2, R17.1
- new net: R18.2, U1.6 (-), U1.7
Changed lines of the file:
@@
 	4600 6500 4700 6500
 Wire Wire Line
-	4700 6500 4700 4550
+	4700 6500 4700 6250
 $Comp
 L Device:R R10
@@
 	1    0    0    -1
 $EndComp
+$Comp
+L Device:R R17
+U 1 1 5FF5423B
+P 5050 5750
+F 0 "R17" V 4843 5750 50  0000 C CNN
+F 1 "470R" V 4934 5750 50  0000 C CNN
+F 2 "Resistor_THT:R_Axial_DIN0207_L6.3mm_D2.5mm_P7.62mm_Horizontal" V 4980 5750 50  0001 C CNN
+F 3 "~" H 5050 5750 50  0001 C CNN
+	1    5050 5750
+	0    1    1    0
+$EndComp
+$Comp
+L Device:C_Small C8
+U 1 1 5FF5C3C7
+P 5500 5750
+F 0 "C8" V 5271 5750 50  0000 C CNN
+F 1 "1nf" V 5362 5750 50  0000 C CNN
+F 2 "Capacitor_THT:C_Disc_D5.0mm_W2.5mm_P5.00mm" H 5500 5750 50  0001 C CNN
+F 3 "~" H 5500 5750 50  0001 C CNN
+	1    5500 5750
+	0    1    1    0
+$EndComp
+$Comp
+L power:GND #PWR05
+U 1 1 5FF6328D
+P 5650 5950
+F 0 "#PWR05" H 5650 5700 50  0001 C CNN
+F 1 "GND" H 5655 5777 50  0000 C CNN
+F 2 "" H 5650 5950 50  0001 C CNN
+F 3 "" H 5650 5950 50  0001 C CNN
+	1    5650 5950
+	1    0    0    -1
+$EndComp
+Wire Wire Line
+	5600 5750 5650 5750
+Wire Wire Line
+	5650 5750 5650 5950
+Wire Wire Line
+	5400 5750 5200 5750
+Wire Wire Line
+	4900 5750 4700 5750
+Connection ~ 4700 5750
+Wire Wire Line
+	4700 5750 4700 4550
+$Comp
+L Device:R R18
+U 1 1 5FF92A35
+P 4700 6100
+F 0 "R18" H 4770 6146 50  0000 L CNN
+F 1 "100K" H 4770 6055 50  0000 L CNN
+F 2 "Resistor_THT:R_Axial_DIN0207_L6.3mm_D2.5mm_P7.62mm_Horizontal" V 4630 6100 50  0001 C CNN
+F 3 "~" H 4700 6100 50  0001 C CNN
+	1    4700 6100
+	1    0    0    -1
+$EndComp
+Wire Wire Line
+	4700 5950 4700 5750
 $EndSCHEMATC

Commit message: three new modules with pcbs
Parts:
- removed J6: Power In, Connector_PinHeader_2.54mm:PinHeader_1x04_P2.54mm_Vertical, symbol Connector:Conn_01x04_Male
- added C9: 10uf, Capacitor_THT:CP_Radial_D5.0mm_P2.00mm, symbol Device:CP
- added J6: Power In, Connector_PinHeader_2.54mm:PinHeader_1x03_P2.54mm_Vertical, symbol Connector:Conn_01x03_Male
- added U4: L7805, Package_TO_SOT_THT:TO-220-3_Vertical, symbol Regulator_Linear:L7805
Connections:
- wire segments 165 -> 172
Changed lines of the file:
@@
 Wire Wire Line
 	5100 2500 5350 2500
-$Comp
-L power:-12V #PWR0101
-U 1 1 5FEEE242
-P 5850 3750
-F 0 "#PWR0101" H 5850 3850 50  0001 C CNN
-F 1 "-12V" H 5865 3923 50  0000 C CNN
-F 2 "" H 5850 3750 50  0001 C CNN
-F 3 "" H 5850 3750 50  0001 C CNN
-	1    5850 3750
-	-1   0    0    1
-$EndComp
 Wire Wire Line
 	5850 3600 5850 3750
@@
 	9250 5300 9250 5500
 $Comp
-L Connector:Conn_01x04_Male J6
-U 1 1 600D0320
-P 7100 5750
-F 0 "J6" H 7208 6031 50  0000 C CNN
-F 1 "Power In" H 7208 5940 50  0000 C CNN
-F 2 "Connector_PinHeader_2.54mm:PinHeader_1x04_P2.54mm_Vertical" H 7100 5750 50  0001 C CNN
-F 3 "~" H 7100 5750 50  0001 C CNN
-	1    7100 5750
-	1    0    0    -1
-$EndComp
-$Comp
 L Device:CP_Small C5
 U 1 1 600D75AE
@@
 	1    0    0    -1
 $EndComp
-$Comp
-L Device:CP_Small C7
-U 1 1 600DE019
-P 7850 6200
-F 0 "C7" H 7762 6154 50  0000 R CNN
-F 1 "10uf" H 7762 6245 50  0000 R CNN
-F 2 "Capacitor_THT:CP_Radial_D5.0mm_P2.00mm" H 7850 6200 50  0001 C CNN
-F 3 "~" H 7850 6200 50  0001 C CNN
-	1    7850 6200
-	-1   0    0    1
-$EndComp
-Wire Wire Line
-	7300 6300 7850 6300
-Wire Wire Line
-	7300 5950 7300 6300
 Wire Wire Line
 	7300 5750 7850 5750
@@
 	7350 5650 7350 5350
 Wire Wire Line
-	7350 5350 7850 5350
-Wire Wire Line
 	7300 5850 7400 5850
 Wire Wire Line
@@
 Wire Wire Line
 	7400 5950 7850 5950
-Wire Wire Line
-	7850 6100 8100 6100
-Wire Wire Line
-	8100 6100 8100 5750
-Wire Wire Line
-	8100 5750 7850 5750
 $Comp
 L power:GND #PWR04
@@
 	0    -1   -1   0
 $EndComp
-Wire Wire Line
-	8100 5750 8200 5750
-Connection ~ 8100 5750
 $Comp
 L power:+12V #PWR01
@@
 Connection ~ 7850 5950
 $Comp
-L power:+5V #PWR03
-U 1 1 60139066
-P 7850 6300
-F 0 "#PWR03" H 7850 6150 50  0001 C CNN
-F 1 "+5V" H 7865 6473 50  0000 C CNN
-F 2 "" H 7850 6300 50  0001 C CNN
-F 3 "" H 7850 6300 50  0001 C CNN
-	1    7850 6300
-	-1   0    0    1
-$EndComp
-Connection ~ 7850 6300
-$Comp
 L power:GND #PWR0107
 U 1 1 601A0CA3
@@
 Wire Wire Line
 	4700 5950 4700 5750
+Wire Wire Line
+	5850 3750 4850 3750
+Wire Wire Line
+	4850 3750 4850 2150
+Wire Wire Line
+	4850 2150 4300 2150
+Connection ~ 4300 2150
+$Comp
+L Regulator_Linear:L7805 U4
+U 1 1 601F7ADF
+P 7650 4800
+F 0 "U4" H 7650 5042 50  0000 C CNN
+F 1 "L7805" H 7650 4951 50  0000 C CNN
+F 2 "Package_TO_SOT_THT:TO-220-3_Vertical" H 7675 4650 50  0001 L CIN
+F 3 "http://www.st.com/content/ccc/resource/technical/document/datasheet/41/4f/b3/b0/12/d4/47/88/CD00000444.pdf/files/CD00000444.pdf/jcr:content/translations/en.CD00000444.pdf" H 7650 4750 50  0001 C CNN
+	1    7650 4800
+	1    0    0    -1
+$EndComp
+Wire Wire Line
+	7850 5750 8200 5750
+$Comp
+L Connector:Conn_01x03_Male J6
+U 1 1 6021325A
+P 7100 5750
+F 0 "J6" H 7208 6031 50  0000 C CNN
+F 1 "Power In" H 7208 5940 50  0000 C CNN
+F 2 "Connector_PinHeader_2.54mm:PinHeader_1x03_P2.54mm_Vertical" H 7100 5750 50  0001 C CNN
+F 3 "~" H 7100 5750 50  0001 C CNN
+	1    7100 5750
+	1    0    0    -1
+$EndComp
+Wire Wire Line
+	7350 5350 7850 5350
+Wire Wire Line
+	7350 4800 7350 5100
+Connection ~ 7350 5350
+$Comp
+L Device:CP_Small C7
+U 1 1 60236C72
+P 7450 5100
+F 0 "C7" V 7675 5100 50  0000 C CNN
+F 1 "10uf" V 7584 5100 50  0000 C CNN
+F 2 "Capacitor_THT:CP_Radial_D5.0mm_P2.00mm" H 7450 5100 50  0001 C CNN
+F 3 "~" H 7450 5100 50  0001 C CNN
+	1    7450 5100
+	0    -1   -1   0
+$EndComp
+Connection ~ 7350 5100
+Wire Wire Line
+	7350 5100 7350 5350
+Wire Wire Line
+	7550 5100 7650 5100
+$Comp
+L Device:CP C9
+U 1 1 6023F4A5
+P 8100 5000
+F 0 "C9" H 8218 5046 50  0000 L CNN
+F 1 "10uf" H 8218 4955 50  0000 L CNN
+F 2 "Capacitor_THT:CP_Radial_D5.0mm_P2.00mm" H 8138 4850 50  0001 C CNN
+F 3 "~" H 8100 5000 50  0001 C CNN
+	1    8100 5000
+	1    0    0    -1
+$EndComp
+Wire Wire Line
+	7950 4800 8100 4800
+Wire Wire Line
+	8100 4800 8100 4850
+Wire Wire Line
+	8100 5150 7650 5150
+Wire Wire Line
+	7650 5150 7650 5100
+Connection ~ 7650 5100
+$Comp
+L power:GND #PWR03
+U 1 1 6024F789
+P 7650 5200
+F 0 "#PWR03" H 7650 4950 50  0001 C CNN
+F 1 "GND" H 7655 5027 50  0000 C CNN
+F 2 "" H 7650 5200 50  0001 C CNN
+F 3 "" H 7650 5200 50  0001 C CNN
+	1    7650 5200
+	1    0    0    -1
+$EndComp
+Wire Wire Line
+	7650 5150 7650 5200
+Connection ~ 7650 5150
+$Comp
+L power:+5V #PWR06
+U 1 1 60257978
+P 8250 4800
+F 0 "#PWR06" H 8250 4650 50  0001 C CNN
+F 1 "+5V" V 8265 4928 50  0000 L CNN
+F 2 "" H 8250 4800 50  0001 C CNN
+F 3 "" H 8250 4800 50  0001 C CNN
+	1    8250 4800
+	0    1    1    0
+$EndComp
+Wire Wire Line
+	8100 4800 8250 4800
+Connection ~ 8100 4800
 $EndSCHEMATC
